File: Hardware/OpenBook_PCB.brd (EAGLE design)
At the start: 175.6 x 111.8 mm, 103 parts, among them IC1 XC6220A331MR-G, IC5 BD5229G-TR, J1 FH34SRJ-24S-0.5SH_99_, J2 SAMACSYS_PARTS_USB4110-GF-A, J3 QWIIC_RIGHT_ANGLE, J4 112A-TAAR-R03_ATTEND, Q1 20V/4.2A/52mΩ/1.4W, Q2 20V/4.2A/52mΩ/1.4W, Q3 SI1308EDL-T1-GE3, U1 W25Q512JVEIQ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

Commit message: Added cutout for PCB near buttons (fixes #7)
Other:
- board size 175.6 x 111.8 mm -> 177.1 x 114.4 mm
Changed lines of the file:
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@@
 <layer number="43" name="vRestrict" color="2" fill="10" visible="yes" active="yes"/>
 <layer number="44" name="Drills" color="7" fill="1" visible="no" active="yes"/>
-<layer number="45" name="Holes" color="7" fill="1" visible="no" active="yes"/>
+<layer number="45" name="Holes" color="7" fill="1" visible="yes" active="yes"/>
 <layer number="46" name="Milling" color="3" fill="1" visible="no" active="yes"/>
 <layer number="47" name="Measures" color="7" fill="1" visible="yes" active="yes"/>
@@
 <dimension x1="83.8" y1="74.4" x2="161.9" y2="75.4" x3="122.85" y3="75.4" textsize="1.778" layer="20" dtype="horizontal" precision="1"/>
 <dimension x1="165.8" y1="75.5" x2="165" y2="119.4" x3="165" y3="97.45" textsize="1.778" layer="20" dtype="vertical" precision="1"/>
-<dimension x1="-12.3" y1="120.5" x2="11.7" y2="120.4" x3="-0.3" y3="120.4" textsize="1.778" layer="20" dtype="horizontal" precision="1"/>
-<dimension x1="-12.9" y1="121.3" x2="36.1" y2="122.3" x3="11.6" y3="122.3" textsize="1.778" layer="20" dtype="horizontal" precision="1"/>
-<dimension x1="-12.8" y1="123.3" x2="51.1" y2="123.1" x3="19.15" y3="123.1" textsize="1.778" layer="20" dtype="horizontal" precision="1"/>
-<dimension x1="-13.2" y1="125.8" x2="79" y2="124.9" x3="32.9" y3="124.9" textsize="1.778" layer="20" dtype="horizontal" precision="1"/>
-<wire x1="15.8" y1="119.05" x2="-12.7" y2="119.05" width="0" layer="20"/>
-<wire x1="-12.7" y1="119.05" x2="-12.7" y2="118.5" width="0" layer="20"/>
+<dimension x1="-11.565" y1="120.451" x2="12.435" y2="120.351" x3="0.435" y3="120.351" textsize="1.778" layer="20" dtype="horizontal" precision="1"/>
+<dimension x1="-11.561" y1="121.12" x2="37.439" y2="122.12" x3="12.939" y3="122.12" textsize="1.778" layer="20" dtype="horizontal" precision="1"/>
+<dimension x1="-11.583" y1="124.346" x2="52.317" y2="124.146" x3="20.367" y3="124.146" textsize="1.778" layer="20" dtype="horizontal" precision="1"/>
+<dimension x1="-11.611" y1="126.688" x2="80.589" y2="125.788" x3="34.489" y3="125.788" textsize="1.778" layer="20" dtype="horizontal" precision="1"/>
+<wire x1="-12.707" y1="119.124" x2="-12.7" y2="118.5" width="0" layer="20"/>
 <wire x1="-12.7" y1="7.62" x2="-12.7" y2="7.5" width="0.1524" layer="20"/>
 <wire x1="-12.7" y1="7.5" x2="74.7544875" y2="7.5" width="0.1524" layer="20"/>
@@
 <wire x1="92.3" y1="17.2" x2="92.3" y2="7.62" width="0.1524" layer="20"/>
 <wire x1="92.3" y1="7.62" x2="162.9" y2="7.62" width="0.1524" layer="20"/>
-<wire x1="84" y1="75.6" x2="84" y2="119.05" width="0.1524" layer="20"/>
-<wire x1="84" y1="75.6" x2="162.9" y2="75.6" width="0.1524" layer="20"/>
+<wire x1="83.929" y1="75.6" x2="83.594" y2="119.206" width="0.1524" layer="20"/>
+<wire x1="83.929" y1="75.6" x2="162.9" y2="75.6" width="0.1524" layer="20"/>
 <wire x1="-5.932" y1="71.838" x2="-5.738" y2="53.432" width="0.1524" layer="20"/>
 <wire x1="-5.738" y1="53.432" x2="-6.038" y2="53.132" width="0.1524" layer="20"/>
@@
 <wire x1="-11.865" y1="53.089" x2="-11.8" y2="7.7" width="0.1524" layer="20"/>
 <wire x1="-11.8" y1="7.7" x2="-12.7" y2="7.5" width="0.1524" layer="20"/>
-<wire x1="84" y1="119.05" x2="15.8" y2="119.05" width="0.1524" layer="20"/>
-<wire x1="15.8" y1="119.05" x2="-11.65" y2="119.35" width="0.1524" layer="20"/>
-<wire x1="-11.65" y1="119.35" x2="-11.582" y2="72.138" width="0.1524" layer="20"/>
+<wire x1="83.594" y1="119.206" x2="56.388" y2="119.355" width="0.1524" layer="20"/>
+<wire x1="-11.226" y1="119.647" x2="-11.582" y2="72.138" width="0.1524" layer="20"/>
 <wire x1="-5.932" y1="71.838" x2="-11.582" y2="72.138" width="0.1524" layer="20"/>
 <wire x1="162.9" y1="75.6" x2="162.9" y2="7.62" width="0.1524" layer="20"/>
 <dimension x1="-12.5" y1="119.2" x2="-14.578" y2="103.944" x3="-14.578" y3="111.572" textsize="1.778" layer="20" dtype="vertical"/>
 <dimension x1="-17.044" y1="119.244" x2="-18.524" y2="75.223" x3="-18.524" y3="97.2335" textsize="1.778" layer="20" dtype="vertical"/>
+<rectangle x1="-14.219" y1="121.585" x2="-13.808" y2="121.877" layer="20"/>
+<wire x1="-11.226" y1="119.647" x2="7.731" y2="119.551" width="0.1524" layer="20"/>
+<wire x1="7.731" y1="119.551" x2="7.765" y2="118.451" width="0.1524" layer="20"/>
+<wire x1="7.765" y1="118.451" x2="56.422" y2="118.451" width="0.1524" layer="20"/>
+<wire x1="56.422" y1="118.451" x2="56.388" y2="119.355" width="0.1524" layer="20"/>
 </plain>
 <attributes>
@@
 <elements>
 <element uuid="2882400121" name="BOOT_BUTTON" library="DeskAssistant v19 v1" library_urn="urn:adsk.wipprod:fs.file:vf.HBQyDAqPQAGgNTqJqZ0RUQ" package="MYBUTTON" value="BUTTON_CUSYOMV1" x="12.73" y="116.759" smashed="yes">
-<attribute name="NAME" x="11.46" y="119.299" size="1.27" layer="25"/>
+<attribute name="NAME" x="-6.334" y="117.212" size="1.27" layer="25"/>
 </element>
 <element uuid="2882400101" name="C1" library="DeskAssistant v19 v1" library_urn="urn:adsk.wipprod:fs.file:vf.HBQyDAqPQAGgNTqJqZ0RUQ" package="ESP32_WROVER_EAGLE-LTSPICE_C0402" value="100nF" x="91.44" y="73.66" smashed="yes">
@@
 <vertex x="83.9160375" y="119.2238"/>
 <vertex x="61.2315625" y="119.2238"/>
-<vertex x="61.1431625" y="119.1354"/>
-<vertex x="61.11515625" y="119.1238"/>
-<vertex x="-11.5638" y="119.1238"/>
+<vertex x="61.0981625" y="119.0904"/>
+<vertex x="61.07015625" y="119.0788"/>
+<vertex x="-11.5638" y="119.0788"/>
 <vertex x="-11.5638" y="71.9822"/>
 <vertex x="-6.08484375" y="71.9822"/>
@@
 <vertex x="84.1238" y="90.3315625"/>
 <vertex x="84.1238" y="119.1684375"/>
-<vertex x="84.0684375" y="119.2238"/>
-<vertex x="74.7315625" y="119.2238"/>
-<vertex x="74.6431625" y="119.1354"/>
-<vertex x="74.61515625" y="119.1238"/>
-<vertex x="-11.3428" y="119.1238"/>
+<vertex x="83.9944375" y="119.2978"/>
+<vertex x="-11.3428" y="119.2978"/>
 <vertex x="-11.3428" y="72.10105625"/>
-<vertex x="-5.890225" y="72.870003125"/>
-<vertex x="-5.88515625" y="72.872103125"/>
-<vertex x="-5.8753375" y="72.872103125"/>
-<vertex x="-5.86563125" y="72.873471875"/>
-<vertex x="-5.860328125" y="72.872103125"/>
-<vertex x="-5.85484375" y="72.872103125"/>
-<vertex x="-5.845775" y="72.868346875"/>
-<vertex x="-5.83628125" y="72.865896875"/>
-<vertex x="-5.831903125" y="72.8626"/>
-<vertex x="-5.8268375" y="72.860503125"/>
-<vertex x="-5.8199" y="72.853565625"/>
-<vertex x="-5.8120625" y="72.847665625"/>
-<vertex x="-5.809278125" y="72.84294375"/>
-<vertex x="-5.8054" y="72.839065625"/>
-<vertex x="-5.801646875" y="72.83000625"/>
-<vertex x="-5.7966625" y="72.821553125"/>
-<vertex x="-5.795896875" y="72.816121875"/>
-<vertex x="-5.7938" y="72.811059375"/>
-<vertex x="-5.7938" y="72.80124375"/>
-<vertex x="-5.79243125" y="72.791534375"/>
-<vertex x="-5.7938" y="72.78623125"/>
+<vertex x="-5.890225" y="72.87"/>
+<vertex x="-5.88515625" y="72.8721"/>
+<vertex x="-5.8753375" y="72.8721"/>
+<vertex x="-5.86563125" y="72.87346875"/>
+<vertex x="-5.860328125" y="72.8721"/>
+<vertex x="-5.85484375" y="72.8721"/>
+<vertex x="-5.845775" y="72.86834375"/>
+<vertex x="-5.83628125" y="72.86589375"/>
+<vertex x="-5.831903125" y="72.862596875"/>
+<vertex x="-5.8268375" y="72.8605"/>
+<vertex x="-5.8199" y="72.8535625"/>
+<vertex x="-5.8120625" y="72.8476625"/>
+<vertex x="-5.809278125" y="72.842940625"/>
+<vertex x="-5.8054" y="72.8390625"/>
+<vertex x="-5.801646875" y="72.830003125"/>
+<vertex x="-5.7966625" y="72.82155"/>
+<vertex x="-5.795896875" y="72.81611875"/>
+<vertex x="-5.7938" y="72.81105625"/>
+<vertex x="-5.7938" y="72.801240625"/>
+<vertex x="-5.79243125" y="72.79153125"/>
+<vertex x="-5.7938" y="72.786228125"/>
 <vertex x="-5.7938" y="53.75284375"/>
 <vertex x="-5.8054" y="53.7248375"/>
